File: hardware/emonPi_v2.0.0.sch (EAGLE design)
At the start: 67 parts, among them IC1 AVR128DB32-I_PT, IC2 MCP1501-10E_SN, J1 SJ-3524-SMT-TR, J2 SJ-3524-SMT-TR, J4 SJ-3524-SMT-TR, J9 RJ11, Y1 MCSJK-7U-12.00-12-10-80-B-10

Commit message: emonPi v2 redesigned to use AVR128DB48++
Parts:
- removed CTRL: KMR2, microbuilder:SWITCH_TACT_SMT4.6X2.8
- removed IC1: AVR128DB32-I_PT, AVR128DB32-I_PT:AVR128DB32-I_PT
- removed IC2: MCP1501-10E_SN, MCP1501-10E_SN:MCP1501-10E_SN
- removed J9: RJ11, SparkFun-Connectors:RJ11-6
- removed JP2: (no value), pinhead:PINHD-1X5
- removed JP3: (no value), pinhead:PINHD-1X4
- removed LED1: Red 1.85V, adafruit:LEDCHIP-LED0805
- removed U$14: RFM12B, JeeParts:RFM12B
- removed X1: (no value), adafruit:SMACONNECTOR
- removed Y1: MCSJK-7U-12.00-12-10-80-B-10, MCSJK-7U-12.00-12-10-80-B-10:MCSJK-7U-12.00-12-10-80-B-10
- added 3V3_LINK, GND_LINK, SL2, SL4: SOLDERJUMPERNC, SparkFun:SOLDERJUMPERNC
- added ANALOG_EXPANDER: (no value), adafruit:PINHD-1X9
- added AVRDB: AVR128DB48T-E_6LX, AVR128DB48T-E_6LX:AVR128DB48T-E_6LX
- added C17: 22pF, resistor:C-EUC0603
- added C18, C20, C21, C22, C24, C25: 100nF, resistor:C-EUC0603
- added C23, C26: 100nF, rcl:C-EUC0603
- added C27, C28: 2.2uF, rcl:C-EUC0603
- added CN1, CN2, CN3: (no value), SparkFun-Connectors:CONN_03SCREW
- added CP2102: CP210X_USB_UART, SparkFun-DigitalIC:CP210X_USB_UART
- added D10, D11, D5, D6, D7, D8, D9: ESD, microbuilder:DIODESOD-523
- added J3, J5, J6: SJ-3524-SMT-TR, SJ-3524-SMT-TR:SJ-3524-SMT-TR
- added JP5, JP6: (no value), adafruit:PINHD-1X13_BIG
- added LED: Red 1.85V, adafruit:LEDCHIP-LED0805
- added MCP1501: MCP1501-10E_SN, MCP1501-10E_SN:MCP1501-10E_SN
- added R18, R19: 33k, rcl:R-EU_R0603
- added R31, R32, R33, R34: 1k, rcl:R-EU_R0603
- added R35, R36, R37, R38, R39, R40: 10k, rcl:R-EU_R0603
- added R41: 120k, rcl:R-EU_R0603
- added R42: 10R, rcl:R-EU_R0603
- added R43: 4K7, rcl:R-EU_R0603
- added RFM69: RFM12B/69CW, eagle_jeelabs:RFM12B/69CW
- added RJ45: RJ45-8PTH, SparkFun-Connectors:RJ45-8PTH
- added SL1, SL3, UART_3.3, USB_RX, USB_TX: JUMPER-SMT_2_NC_PASTE_NO-SILK, SparkFun-Jumpers:JUMPER-SMT_2_NC_PASTE_NO-SILK
- added SMA: (no value), adafruit:SMACONNECTOR
- added USB-C: CSP-USC16-TR, CSP-USC16-TR:CSP-USC16-TR
- added XTAL: MCSJK-7U-12.00-12-10-80-B-10, MCSJK-7U-12.00-12-10-80-B-10:MCSJK-7U-12.00-12-10-80-B-10
- C10: value 2.2uF -> 10uF 6V
- C11: value 100nF -> 1uF 6V; device rcl:C-EUC0603 -> resistor:C-EUC0603
- C12: value 10uF -> 1uF 6V; device rcl:C-EUC0603 -> resistor:C-EUC0603
- C15: value 100nF -> 1uF 6V
- C16: value 10uF 6V -> 22pF
- C4, C5: value 100nF -> 10uF 6V; device rcl:C-EUC0603 -> resistor:C-EUC0603
- C6: value 100nF -> 10uF 6V
- C7, C8: value 22pF -> 10uF 6V
- C9: value 2.2uF -> 10uF 6V; device rcl:C-EUC0603 -> resistor:C-EUC0603
- D1, D2, D3: value ESD5Z3.3T1G -> ESD
- JP1: value (none) -> 6x1; device pinhead:PINHD-2X6 -> SparkFun:FTDI_BASICPTH
- OLED: device con-lstb-db:MA04-1-OLEDOLED -> con-lstb-db:MA04-1-OLED
- R1, R2, R3: value (none) -> 1M
- R10, R11, R12: value 33k -> 180k
- R13, R14, R15: value 1k -> 180k
- R16, R20, R22, R23: value 10k -> 33k
- R17: value 1K -> 33k
- R21: value 10R -> 33k
- R24: value 4K7 -> 33k
- R25: value 120K -> 1k
- R26, R28: value 10K -> 1k
- R27: value 1K -> 1k
- R29: value 180k -> 1k
- R30: value 33k -> 1k
- R4, R5, R6: value (none) -> 1M; device rcl:R-EU_0204/7 -> rcl:R-EU_R1206
Connections:
- removed net CONTROL: CTRL.P, CTRL.P1, JP1.11, R28.2, S1.NO_1, S1.NO_2
- removed net PULSE_INPUT: IC1.PF3, JP3.3
- removed net _CT1: C1.1, J1.TIP, R1.2, R4.2
- removed net _CT2: C2.1, J2.TIP, R2.2, R5.2
- removed net _CT3: C3.1, J4.TIP, R3.2, R6.2
- new net CT10: ANALOG_EXPANDER.6, AVRDB.PF1_(XTAL32K2)
- new net CT11: ANALOG_EXPANDER.5, AVRDB.PF2
- new net CT4: AVRDB.PD6, D4.C, R28.1
- new net CT5: AVRDB.PE0, D5.C, R29.1
- new net CT6: AVRDB.PE1, D6.C, R30.1
- new net CT7: ANALOG_EXPANDER.9, AVRDB.PE2
- new net CT8: ANALOG_EXPANDER.8, AVRDB.PE3
- new net CT9: ANALOG_EXPANDER.7, AVRDB.PF0_(XTAL32K1)
- new net D+: CP2102.D+, D11.C, USB-C.D1+
- new net D-: CP2102.D-, D10.C, USB-C.D1-
- new net DTR: C26.1, CP2102.DTR
- new net LCD_BUTTON: JP6.4, R39.2, S1.COM_1, S1.NO_1
- new net N$1: C1.1, J1.TIP, R1.2
- new net N$12: C9.2, R15.1, R24.2, R33.2
- new net N$13: C2.1, J2.TIP, R2.2
- new net N$17: C4.2, R10.1, R19.1, R28.2
- new net N$19: C6.1, J6.TIP, R6.2
- new net N$20: C6.2, R12.1, R21.1, R30.2
- new net N$22: CN1.2, SL1.2, SL2.2
- new net N$23: CN2.2, SL3.2, SL4.2
- new net N$24: GND_LINK.2, RJ45.6
- new net N$25: AP2112.EN, R40.2
- new net N$26: C28.1, R37.2, R42.1
- new net N$28: 3V3_LINK.2, JP6.1
- new net N$3: C3.1, J3.TIP, R3.2
- new net N$31: C25.2, CP2102.VDD
- new net N$33: JP1.5, UART_3.3.2
- new net N$4: C8.2, R14.1, R23.2, R32.2
- new net N$5: C4.1, J4.TIP, R4.2
- new net PULSE1: AVRDB.PB5, JP6.7, SL4.1
- new net PULSE2: AVRDB.PC0, JP6.8, SL2.1
- new net RFM_IRQ: JP5.11, RFM69.DIO0/IRQ
- new net RFM_RESET: JP5.12, RFM69.RST
- new net USB_RXD: CP2102.RXD, USB_RX.1
- new net USB_TXD: CP2102.TXD, USB_TX.1
- net +5V: now also C14.2, C24.2, CP2102.REGIN, CP2102.VBUS, JP5.1, JP5.2, R40.1, RJ45.4, RJ45.5, USB-C.VBUS1; no longer C13.2, J9.2, JP1.2, R26.1
- net 3.3V: now also 3V3_LINK.1, ANALOG_EXPANDER.2, AVRDB.AVDD, AVRDB.VDD, AVRDB.VDDIO2, C10.1, C13.1, C18.1, C19.1, C20.1, C21.2, C23.1, C27.1, CN1.3, CN2.3, CN3.3, MCP1501.SHDN, MCP1501.VDD, R10.2, R11.2, R12.2, R13.2, R14.2, R15.2, R35.2, R39.1, R41.2, R43.1, RFM69.VCC, UART_3.3.1; no longer C14.2, C4.1, C5.2, C6.1, C9.1, IC1.AVDD, IC1.VDD, IC1.VDDIO2, IC2.SHDN, IC2.VDD, JP2.1, JP3.1, R16.2, R24.1, R25.2, R28.1, R29.2, U$14.VCC
- net ANALOG_INPUT: now also ANALOG_EXPANDER.4, AVRDB.PF3, CN3.2; no longer IC1.PF4
- net AVR_RX: now also AVRDB.PB1, JP1.3, JP5.4, USB_TX.2; no longer IC1.PC1, JP1.8
- net AVR_TX: now also AVRDB.PB0, JP1.2, JP5.5, USB_RX.2; no longer IC1.PC0, JP1.10
- net CT1: now also AVRDB.PD3, R25.2; no longer IC1.PD3, R13.2
- net CT2: now also AVRDB.PD4, R26.2; no longer IC1.PD2, R14.2
- net CT3: now also AVRDB.PD5, R27.1; no longer IC1.PD1, R15.1
- net DIG1: now also RFM69.ANT, SMA.ANT; no longer U$14.ANT, X1.ANT
- net DS18B20: now also AVRDB.PB4, JP6.6, R43.2, SL1.1, SL3.1; no longer IC1.PA2, JP1.12, JP3.2, R24.2
- net GND: now also ANALOG_EXPANDER.1, AVRDB.EP, AVRDB.GND_1, AVRDB.GND_2, AVRDB.GND_3, C13.2, C16.1, C17.2, C18.2, C19.2, C20.2, C21.1, C23.2, C24.1, C25.1, C27.2, C28.2, CN1.1, CN2.1, CN3.1, CP2102.GND, CP2102.GND@EXP, CP2102.GND@M, D10.A, D11.A, D5.A, D6.A, D7.A, D8.A, D9.A, GND_LINK.1, J3.SLEEVE, J3.TIP_SWITCH, J5.SLEEVE, J5.TIP_SWITCH, J6.SLEEVE, J6.TIP_SWITCH, JP5.10, JP5.3, JP5.7, JP6.5, LED.C, MCP1501.GND_1, MCP1501.GND_2, MCP1501.GND_3, MCP1501.NC, R16.2, R17.2, R18.2, R19.2, R20.2, R21.2, R22.2, R24.1, R36.1, R38.1, RFM69.GND, RFM69.GND1, RJ45.7, RJ45.8, S1.NO_2, SMA.GND1, SMA.GND2, SMA.GND3, SMA.GND4, USB-C.GND1, USB-C.GND2, USB-C.SHIELD, XTAL.GND_1, XTAL.GND_2; no longer C13.1, C4.2, C5.1, C6.2, C7.1, C8.2, C9.2, CTRL.S, CTRL.S1, IC1.GND_1, IC1.GND_2, IC2.GND_1, IC2.GND_2, IC2.GND_3, IC2.NC, J9.1, JP1.9, JP2.5, JP3.4, LED1.C, R10.2, R11.2, R12.2, R20.1, R30.2, S1.COM_1, U$14.GND, X1.GND1, X1.GND2, X1.GND3, X1.GND4, Y1.GND_1, Y1.GND_2
- net LED: now also AVRDB.PC2, R34.2; no longer IC1.PA3, R27.2
- net N$14: now also C5.1, J5.TIP, R5.2; no longer C10.1, R21.1, R22.2
- net N$15: now also C5.2, R11.1, R20.1, R29.2; no longer AP2112.EN, R26.2
- net N$16: now also R17.1, R26.1; no longer R11.1, R14.1
- net N$18: now also R16.1, R25.1; no longer R10.1, R13.1
- net N$2: now also C7.2, R13.1, R22.1, R31.2; no longer C16.2, R17.2, R29.1, R30.1
- net N$21: now also R18.1, R27.2; no longer R12.1, R15.2
- net N$27: now also MCP1501.FEEDBACK, MCP1501.OUT, R36.2, R42.2; no longer IC2.FEEDBACK, IC2.OUT, R20.2, R21.2
- net N$41: now also LED.A, R34.1; no longer LED1.A, R27.1
- net RESET: now also AVRDB.PF6, C22.2, C26.2, R35.1; no longer C19.2, IC1.PF6, R16.1
- net RFM_MISO: now also AVRDB.PA5, JP6.11, RFM69.SDO; no longer IC1.PA5, U$14.SDO
- net RFM_MOSI: now also AVRDB.PA4, JP6.10, RFM69.SDI; no longer IC1.PA4, U$14.SDI
- net RFM_SCK: now also AVRDB.PA6, JP6.12, RFM69.SCK; no longer IC1.PA6, U$14.SCK
- net RFM_SEL: now also AVRDB.PA7, JP5.8, R41.1, RFM69.SEL; no longer IC1.PA7, R25.1, U$14.SEL
- net SCL: now also AVRDB.PB3, JP6.3; no longer IC1.PC3, JP1.5, JP2.3
- net SDA: now also AVRDB.PB2, JP6.2; no longer IC1.PC2, JP1.3, JP2.2
- net UDPI: now also AVRDB.UPDI; no longer IC1.UPDI
- net VREFA: now also ANALOG_EXPANDER.3, AVRDB.PD7, R37.1, R38.2; no longer IC1.PD7, R22.1, R23.2
- net VS1: now also C7.1, RJ45.1; no longer C16.1, J9.6
- net VS2: now also C8.1, RJ45.2; no longer J9.5
- net VS3: now also C9.1, RJ45.3; no longer J9.4
- net VSENS1: now also AVRDB.PD0, D7.C, R31.1; no longer D4.C, IC1.PD6, R17.1
- net VSENS2: now also AVRDB.PD1, D8.C, R32.1; no longer IC1.PD5
- net VSENS3: now also AVRDB.PD2, D9.C, R33.1; no longer IC1.PD4
- net XTAL1: now also AVRDB.PA0_(XTALHF1), C16.2, XTAL.CRYSTAL_1; no longer C7.2, IC1.PA0_(XTALHF1), Y1.CRYSTAL_1
- net XTAL2: now also AVRDB.PA1_(XTALHF2), C17.1, XTAL.CRYSTAL_2; no longer C8.1, IC1.PA1_(XTALHF2), Y1.CRYSTAL_2
- net _RESET: now also C22.1, JP1.1, JP5.6; no longer C19.1, JP1.7
Other:
- note added: "1M Burden resistors not populated Correct values should be choosen if using current output CT sensors."
- note added: "CT Current Sensors"
- note added: "Design is provided "AS IS" and "WITH ALL FAULTS. OpenEnergyMonitor DISCLAIMS ALL OTHER WARRANTIES, EXPRESS OR IMPLIED,"
- note added: "Hardware design files are licensed under the Creative Commons Attribution-ShareAlike 3.0 Unported License"
- note added: "OpenEnergyMonitor.org"
- note added: "Temperature & AC Voltage Sensors"
- note added: "Trystan Lea & Glyn Hudson - March 2022"
- note added: "emonPi2"
- note removed: "One-Wire RJ45"
- moved on the sheet: AP2112, C1, C10, C11, C12, C13, C14, C15, C16, C19, C2, C3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

Commit message: export
Parts:
- added FD1, FD2, FD3: FIDUCIAL1X2, SparkFun-Aesthetics:FIDUCIAL1X2
- added LOGO1: OSHW-LOGOS-COPPER, SparkFun-Aesthetics:OSHW-LOGOS-COPPER
Changed lines of the file:
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@@
 <setting verticaltext="up"/>
 </settings>
-<grid distance="0.05" unitdist="inch" unit="inch" style="lines" multiple="1" display="no" altdistance="0.01" altunitdist="inch" altunit="inch"/>
+<grid distance="0.1" unitdist="inch" unit="inch" style="lines" multiple="1" display="no" altdistance="0.01" altunitdist="inch" altunit="inch"/>
 <layers>
 <layer number="1" name="Top" color="4" fill="1" visible="no" active="no"/>
@@
 <part name="P+2" library="SparkFun" deviceset="3.3V" device=""/>
 <part name="UART_3.3" library="SparkFun-Jumpers" deviceset="JUMPER-SMT_2_NC_PASTE" device="_NO-SILK" package3d_urn="urn:adsk.eagle:package:39283/1"/>
+<part name="FD1" library="SparkFun-Aesthetics" deviceset="FIDUCIAL" device="1X2"/>
+<part name="FD2" library="SparkFun-Aesthetics" deviceset="FIDUCIAL" device="1X2"/>
+<part name="FD3" library="SparkFun-Aesthetics" deviceset="FIDUCIAL" device="1X2"/>
+<part name="LOGO1" library="SparkFun-Aesthetics" deviceset="OSHW-LOGO" device="S-COPPER"/>
 </parts>
 <sheets>
@@
 <attribute name="NAME" x="300.99" y="286.766" size="1.9304" layer="95" font="vector" align="center"/>
 </instance>
+<instance part="FD1" gate="G$1" x="408.94" y="246.38" smashed="yes"/>
+<instance part="FD2" gate="G$1" x="408.94" y="241.3" smashed="yes"/>
+<instance part="FD3" gate="G$1" x="408.94" y="236.22" smashed="yes"/>
+<instance part="LOGO1" gate="G$1" x="388.62" y="241.3" smashed="yes"/>
 </instances>
 <busses>
