File: hardware/fascias_v2.0.0.brd (EAGLE design)
At the start: 154.7 x 183.2 mm, 0 parts

Commit message: updated fascia
Other:
- board size 154.7 x 183.2 mm -> 173.5 x 231.2 mm
Changed lines of the file:
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@@
 <setting verticaltext="up"/>
 </settings>
-<grid distance="0.01" unitdist="mm" unit="mm" style="lines" multiple="1" display="yes" altdistance="0.005" altunitdist="inch" altunit="inch"/>
+<grid distance="1" unitdist="mm" unit="mm" style="lines" multiple="1" display="yes" altdistance="0.005" altunitdist="inch" altunit="inch"/>
 <layers>
-<layer number="1" name="Top" color="4" fill="1" visible="no" active="yes"/>
+<layer number="1" name="Top" color="4" fill="1" visible="yes" active="yes"/>
 <layer number="16" name="Bottom" color="1" fill="1" visible="no" active="yes"/>
 <layer number="17" name="Pads" color="2" fill="1" visible="no" active="yes"/>
@@
 <wire x1="1.3" y1="4.3" x2="1.3" y2="41.5" width="0.15" layer="20"/>
 <circle x="14" y="32.5" radius="3.04138125" width="0.15" layer="20"/>
-<wire x1="13" y1="10" x2="68" y2="10" width="0.15" layer="20"/>
-<wire x1="68" y1="10" x2="68" y2="27" width="0.15" layer="20"/>
-<wire x1="68" y1="27" x2="13" y2="27" width="0.15" layer="20"/>
-<wire x1="13" y1="27" x2="13" y2="10" width="0.15" layer="20"/>
 <circle x="12" y="84.5" radius="3.5" width="0.15" layer="20"/>
 <wire x1="45.5" y1="78" x2="56.5" y2="78" width="0.15" layer="20"/>
@@
 <wire x1="60.5" y1="58" x2="46.5" y2="58" width="0.15" layer="20"/>
 <wire x1="46.5" y1="58" x2="46.5" y2="54" width="0.15" layer="20"/>
-<wire x1="2" y1="99" x2="76" y2="99" width="0.15" layer="20"/>
-<wire x1="2" y1="99" x2="2" y2="184" width="0.15" layer="20"/>
-<wire x1="2" y1="184" x2="76" y2="184" width="0.15" layer="20"/>
-<wire x1="76" y1="99" x2="76" y2="184" width="0.15" layer="20"/>
-<circle x="40.622" y="117.022" radius="3" width="0.15" layer="20"/>
-<wire x1="82" y1="99" x2="156" y2="99" width="0.15" layer="20"/>
-<wire x1="82" y1="99" x2="82" y2="184" width="0.15" layer="20"/>
-<wire x1="82" y1="184" x2="156" y2="184" width="0.15" layer="20"/>
-<wire x1="156" y1="99" x2="156" y2="184" width="0.15" layer="20"/>
+<wire x1="10" y1="98" x2="84" y2="98" width="0.15" layer="20"/>
+<wire x1="10" y1="98" x2="10" y2="183" width="0.15" layer="20"/>
+<wire x1="10" y1="183" x2="84" y2="183" width="0.15" layer="20"/>
+<wire x1="84" y1="98" x2="84" y2="183" width="0.15" layer="20"/>
+<circle x="43.5" y="114.5" radius="3" width="0.15" layer="20"/>
+<wire x1="100.79" y1="99" x2="174.79" y2="99" width="0.15" layer="20"/>
+<wire x1="100.79" y1="99" x2="100.79" y2="184" width="0.15" layer="20"/>
+<wire x1="100.79" y1="184" x2="174.79" y2="184" width="0.15" layer="20"/>
+<wire x1="174.79" y1="99" x2="174.79" y2="184" width="0.15" layer="20"/>
 <circle x="4.86" y="89.6" radius="1.7" width="0.15" layer="20"/>
 <circle x="89.18" y="89.57" radius="1.7" width="0.15" layer="20"/>
@@
 <circle x="89.19" y="4.36" radius="1.7" width="0.15" layer="20"/>
 <circle x="89.19" y="41.57" radius="1.7" width="0.15" layer="20"/>
+<wire x1="13" y1="26" x2="14" y2="27" width="0.1524" layer="20" curve="-90"/>
+<wire x1="68" y1="11" x2="67" y2="10" width="0.1524" layer="20" curve="-90"/>
+<wire x1="67" y1="27" x2="68" y2="26" width="0.1524" layer="20" curve="-90"/>
+<wire x1="14" y1="10" x2="13" y2="11" width="0.1524" layer="20" curve="-90"/>
+<wire x1="14" y1="27" x2="67" y2="27" width="0.1524" layer="20"/>
+<wire x1="68" y1="26" x2="68" y2="11" width="0.1524" layer="20"/>
+<wire x1="67" y1="10" x2="14" y2="10" width="0.1524" layer="20"/>
+<wire x1="13" y1="11" x2="13" y2="26" width="0.1524" layer="20"/>
+<wire x1="89.6" y1="-2.9" x2="93.2" y2="-6.4" width="0.15" layer="20" curve="-90"/>
+<wire x1="93.2" y1="-43.6" x2="89.6" y2="-47.2" width="0.15" layer="20" curve="-90"/>
+<wire x1="93.2" y1="-43.6" x2="93.2" y2="-6.4" width="0.15" layer="20"/>
+<wire x1="89.6" y1="-2.9" x2="5.3" y2="-2.9" width="0.15" layer="20"/>
+<wire x1="89.6" y1="-47.2" x2="5.4" y2="-47.2" width="0.15" layer="20"/>
+<wire x1="1.8" y1="-6.5" x2="5.3" y2="-2.9" width="0.15" layer="20" curve="-90"/>
+<wire x1="5.4" y1="-47.2" x2="1.8" y2="-43.7" width="0.15" layer="20" curve="-90"/>
+<wire x1="1.8" y1="-43.7" x2="1.8" y2="-6.5" width="0.15" layer="20"/>
+<circle x="14.5" y="-15.5" radius="3.04138125" width="0.15" layer="20"/>
+<circle x="27.5" y="-15.5" radius="3.04138125" width="0.15" layer="20"/>
+<circle x="40.5" y="-15.5" radius="3.04138125" width="0.15" layer="20"/>
+<circle x="54.5" y="-15.5" radius="3.04138125" width="0.15" layer="20"/>
+<circle x="67.5" y="-15.5" radius="3.04138125" width="0.15" layer="20"/>
+<circle x="80.5" y="-15.5" radius="3.04138125" width="0.15" layer="20"/>
+<circle x="5.37" y="-6.43" radius="1.7" width="0.15" layer="20"/>
+<circle x="5.36" y="-43.65" radius="1.7" width="0.15" layer="20"/>
+<circle x="89.69" y="-43.64" radius="1.7" width="0.15" layer="20"/>
+<circle x="89.69" y="-6.43" radius="1.7" width="0.15" layer="20"/>
+<circle x="14.5" y="-26.7" radius="3.04138125" width="0.15" layer="20"/>
+<circle x="27.5" y="-26.7" radius="3.04138125" width="0.15" layer="20"/>
+<circle x="40.5" y="-26.7" radius="3.04138125" width="0.15" layer="20"/>
+<circle x="54.5" y="-26.7" radius="3.04138125" width="0.15" layer="20"/>
+<circle x="67.5" y="-26.7" radius="3.04138125" width="0.15" layer="20"/>
+<circle x="80.5" y="-26.7" radius="3.04138125" width="0.15" layer="20"/>
 </plain>
 <attributes>
